Commit message: New update, new project it looks amazing !!!

File: prop_arm_description/models/prop_arm/urdf/prop_arm.urdf.xacro (robot description, xacro)
@@ -1,27 +1,32 @@
-<robot name="prop_arm" version="1.0">
-  <joint name="arm.001_link_joint" type="revolute">
-    <limit lower="-3.14000" upper="3.14000" effort="0.00000" velocity="0.00000"/>
-    <origin rpy="-0.00000 1.57080 0.00000" xyz="0.43129 -0.58144 0.11764"/>
-    <parent link="table_link"/>
-    <child link="arm.001_link"/>
-    <axis xyz="0.00000 0.00000 -1.00000"/>
-  </joint>
-  <joint name="motor.001_link_joint" type="fixed">
-    <origin rpy="1.57080 -1.57080 0.00000" xyz="0.40028 -0.03651 0.02656"/>
-    <parent link="arm.001_link"/>
-    <child link="motor.001_link"/>
-  </joint>
-  <joint name="prop_link_joint" type="revolute">
-    <limit lower="-3.14000" upper="3.14000" effort="0.00000" velocity="0.00000"/>
-    <origin rpy="0.00000 0.00000 0.00000" xyz="0.00004 -0.00000 0.02475"/>
-    <parent link="motor.001_link"/>
-    <child link="prop_link"/>
-    <axis xyz="0.00000 0.00000 1.00000"/>
-  </joint>
-  <link name="arm.001_link">
-    <collision name="arm.001_collision">
+<?xml version="1.0" encoding="utf-8"?>
+<robot xmlns:xacro="http://www.ros.org/wiki/xacro" name="prop_arm">
+  <!-- World link -->
+  <link name="world"/>
+  <!-- Main robot link -->
+  <link name="base_link">
+    <collision name="base_collision">
+      <origin rpy="0.00000 0.00000 0.00000" xyz="0.00000 0.00000 0.00000"/>
+      <geometry>
+        <mesh filename="package://prop_arm_description/models/prop_arm/meshes/collisions/base.stl" scale="1.00000 1.00000 1.00000"/>
+      </geometry>
+    </collision>
+    <inertial>
+      <inertia ixx="4.49421" ixy="1.19011" ixz="-0.32403" iyy="1.83979" iyz="0.67570" izz="5.09395"/>
+      <origin rpy="0.00000 0.00000 0.00000" xyz="-0.00341 -0.01201 -0.10842"/>
+      <mass value="10.00000"/>
+    </inertial>
+    <visual name="base">
+      <origin rpy="0.00000 0.00000 0.00000" xyz="0.00000 0.00000 0.00000"/>
+      <geometry>
+        <mesh filename="package://prop_arm_description/models/prop_arm/meshes/visuals/base.dae" scale="1.00000 1.00000 1.00000"/>
+      </geometry>
+    </visual>
+  </link>
+  <!-- Arm link -->
+  <link name="arm_link">
+    <collision name="arm_collision">
       <origin rpy="0.00000 -1.57080 0.00000" xyz="0.00000 0.00000 -0.00000"/>
       <geometry>
-        <mesh filename="../meshes/stl/arm.004.stl" scale="1.00000 1.00000 1.00000"/>
+        <mesh filename="package://prop_arm_description/models/prop_arm/meshes/collisions/arm.stl" scale="1.00000 1.00000 1.00000"/>
       </geometry>
     </collision>
@@ -31,17 +36,17 @@
       <mass value="10.00000"/>
     </inertial>
-    <visual name="arm.001">
+    <visual name="arm">
       <origin rpy="0.00000 -1.57080 0.00000" xyz="0.00000 -0.00000 -0.00000"/>
-      <material name="Material.012"/>
       <geometry>
-        <mesh filename="../meshes/stl/arm.004.stl" scale="1.00000 1.00000 1.00000"/>
+        <mesh filename="package://prop_arm_description/models/prop_arm/meshes/visuals/arm.dae" scale="1.00000 1.00000 1.00000"/>
       </geometry>
     </visual>
   </link>
-  <link name="motor.001_link">
-    <collision name="motor.001_collision">
+  <!-- Motor link -->
+  <link name="motor_link">
+    <collision name="motor_collision">
       <origin rpy="0.00000 0.00000 0.00000" xyz="-0.00000 -0.00000 0.00000"/>
       <geometry>
-        <mesh filename="../meshes/stl/arm.005.stl" scale="1.00000 1.00000 1.00000"/>
+        <mesh filename="package://prop_arm_description/models/prop_arm/meshes/collisions/motor.stl" scale="1.00000 1.00000 1.00000"/>
       </geometry>
     </collision>
@@ -51,17 +56,17 @@
       <mass value="10.00000"/>
     </inertial>
-    <visual name="motor.001">
+    <visual name="motor">
       <origin rpy="0.00000 0.00000 0.00000" xyz="0.00000 0.00000 0.00000"/>
-      <material name="Material.015"/>
       <geometry>
-        <mesh filename="../meshes/stl/arm.005.stl" scale="1.00000 1.00000 1.00000"/>
+        <mesh filename="package://prop_arm_description/models/prop_arm/meshes/visuals/motor.dae" scale="1.00000 1.00000 1.00000"/>
       </geometry>
     </visual>
   </link>
+  <!-- Propeller link-->
   <link name="prop_link">
     <collision name="prop_collision">
       <origin rpy="-0.00000 0.00000 0.00000" xyz="0.00000 0.00000 0.00000"/>
       <geometry>
-        <mesh filename="../meshes/stl/arm.001.stl" scale="1.00000 1.00000 1.00000"/>
+        <mesh filename="package://prop_arm_description/models/prop_arm/meshes/collisions/prop.stl" scale="1.00000 1.00000 1.00000"/>
       </geometry>
     </collision>
@@ -73,41 +78,42 @@
     <visual name="prop">
       <origin rpy="0.00000 0.00000 0.00000" xyz="-0.00000 -0.00000 0.00000"/>
-      <material name="Material.014"/>
       <geometry>
-        <mesh filename="../meshes/stl/arm.001.stl" scale="1.00000 1.00000 1.00000"/>
+        <mesh filename="package://prop_arm_description/models/prop_arm/meshes/visuals/prop.dae" scale="1.00000 1.00000 1.00000"/>
       </geometry>
     </visual>
   </link>
-  <link name="table_link">
-    <collision name="table_collision">
-      <origin rpy="0.00000 0.00000 0.00000" xyz="0.00000 0.00000 0.00000"/>
-      <geometry>
-        <mesh filename="../meshes/stl/arm.stl" scale="1.00000 1.00000 1.00000"/>
-      </geometry>
-    </collision>
-    <inertial>
-      <inertia ixx="4.49421" ixy="1.19011" ixz="-0.32403" iyy="1.83979" iyz="0.67570" izz="5.09395"/>
-      <origin rpy="0.00000 0.00000 0.00000" xyz="-0.00341 -0.01201 -0.10842"/>
-      <mass value="10.00000"/>
-    </inertial>
-    <visual name="table">
-      <origin rpy="0.00000 0.00000 0.00000" xyz="0.00000 0.00000 0.00000"/>
-      <material name="Material.011"/>
-      <geometry>
-        <mesh filename="../meshes/stl/arm.stl" scale="1.00000 1.00000 1.00000"/>
-      </geometry>
-    </visual>
-  </link>
-  <material name="Material.011">
-    <color rgba="0.17255 0.06667 0.01176 1.00000"/>
-  </material>
-  <material name="Material.012">
-    <color rgba="0.16078 0.16078 0.16078 1.00000"/>
-  </material>
-  <material name="Material.014">
-    <color rgba="0.00000 0.00000 0.00000 1.00000"/>
-  </material>
-  <material name="Material.015">
-    <color rgba="0.80000 0.00000 0.00000 1.00000"/>
-  </material>
+  <!-- Joint between world and base -->
+  <joint name="world_base_joint" type="fixed">
+    <parent link="world"/>
+    <child link="base_link"/>
+  </joint>
+  <!-- Joint between base and arm -->
+  <joint name="arm_link_joint" type="continuous">
+    <axis xyz="0 0 -1"/>
+    <origin rpy="0 1.57080 0" xyz="0.43129 -0.58144 0.11764"/>
+    <limit effort="1500.0" velocity="10.0"/>
+    <dynamics damping="0.8" friction="0.3"/>
+    <parent link="base_link"/>
+    <child link="arm_link"/>
+  </joint>
+  <!-- Joint between arm and motor -->
+  <joint name="motor_link_joint" type="fixed">
+    <origin rpy="1.57080 -1.57080 0.00000" xyz="0.40028 -0.03651 0.02656"/>
+    <parent link="arm_link"/>
+    <child link="motor_link"/>
+  </joint>
+  <!-- Joint between motor and propeller -->
+  <joint name="prop_link_joint" type="continuous">
+    <dynamics damping="0.01"/>
+    <origin rpy="0 0 0" xyz="0.00004 0 0.02475"/>
+    <parent link="motor_link"/>
+    <child link="prop_link"/>
+    <axis xyz="0 0 1"/>
+  </joint>
+  <!-- Include materials for Gazebo -->
+  <xacro:include filename="$(find prop_arm_gazebo)/urdf/prop_arm_materials.xacro"/>
+  <!-- Include gazebo plugins -->
+  <xacro:include filename="$(find prop_arm_gazebo_plugins)/urdf/prop_arm_gazebo_plugins.xacro"/>
+  <!-- Include control interface -->
+  <xacro:include filename="$(find prop_arm_gazebo_control)/urdf/prop_arm_control.xacro"/>
 </robot>

Commit message: Enhance prop_arm_gazebo_control with new controllers and improved functionality
- Updated URDF configuration to include new command interfaces for effort, velocity, and position control.
- Added new YAML configuration for motor force controller, including joint state broadcaster and various control types.
- Implemented MotorCommander class for commanding motor actions (angle, force, velocity) with detailed logging and usage instructions.
- Developed PropellerForceController class with PID control for stabilizing the arm at a target angle, including diagnostics and control loops.
- Introduced compatibility with legacy topics while ensuring new controller commands are published correctly.
- Enhanced logging for better debugging and user feedback during operation.

File: prop_arm_description/models/prop_arm/urdf/prop_arm.urdf.xacro (robot description, xacro)
@@ -32,7 +32,7 @@
     </collision>
     <inertial>
-      <inertia ixx="0.45780" ixy="-0.00003" ixz="-0.00533" iyy="0.45909" iyz="-0.00314" izz="0.00510"/>
+      <inertia ixx="0.9156" ixy="-0.00006" ixz="-0.01066" iyy="0.91818" iyz="-0.00628" izz="0.01020"/>
       <origin rpy="0.00000 0.00000 0.00000" xyz="0.14437 -0.00020 0.01985"/>
-      <mass value="10.00000"/>
+      <mass value="20.0"/>
     </inertial>
     <visual name="arm">
@@ -89,9 +89,9 @@
   </joint>
   <!-- Joint between base and arm -->
-  <joint name="arm_link_joint" type="continuous">
+  <joint name="arm_link_joint" type="revolute">
     <axis xyz="0 0 -1"/>
     <origin rpy="0 1.57080 0" xyz="0.43129 -0.58144 0.11764"/>
-    <limit effort="1500.0" velocity="10.0"/>
-    <dynamics damping="0.8" friction="0.3"/>
+    <limit lower="1.5708" upper="3.14159" effort="1500.0" velocity="10.0"/>
+    <dynamics damping="0.0" friction="0.0"/>
     <parent link="base_link"/>
     <child link="arm_link"/>

File: prop_arm_gazebo_control/urdf/prop_arm_control.xacro (robot description, xacro)
@@ -1,8 +1,10 @@
 <?xml version="1.0"?>
 <robot xmlns:xacro="http://www.ros.org/wiki/xacro" name="prop_arm_control">
-    <!-- Gazebo plugin para ros2_control -->
+    <!-- Gazebo plugin for ros2_control -->
     <gazebo>
-        <plugin name="gz_ros2_control::GazeboSimROS2ControlPlugin" filename="libgz_ros2_control-system.so">
-            <parameters>$(find prop_arm_gazebo_control)/config/ros2_controllers.yaml</parameters>
+        <plugin filename="gz_ros2_control-system" name="gz_ros2_control::GazeboSimROS2ControlPlugin">
+            <parameters>$(find prop_arm_gazebo_control)/config/ros2_controllers_motor_force.yaml</parameters>
+            <robot_param>robot_description</robot_param>
+            <robot_param_node>robot_state_publisher</robot_param_node>
         </plugin>
     </gazebo>
@@ -13,11 +15,25 @@
             <param name="robot_namespace">prop_arm</param>
         </hardware>
+        <!-- Define the joint that will be controlled -->
         <joint name="arm_link_joint">
+            <!-- Command interface for direct force/thrust control -->
+            <command_interface name="effort">
+                <param name="min">-100.0</param>
+                <param name="max">100.0</param>
+            </command_interface>
+            <!-- Command interface for direct velocity control -->
+            <command_interface name="velocity">
+                <param name="min">-785.0</param>
+                <param name="max">785.0</param>
+            </command_interface>
+            <!-- Command interface for position control (angle control) -->
             <command_interface name="position">
-                <param name="min">-6.28</param>
-                <param name="max">6.28</param>
+                <param name="min">-3.14159</param>
+                <param name="max">3.14159</param>
             </command_interface>
+            <!-- State interfaces -->
             <state_interface name="position"/>
             <state_interface name="velocity"/>
+            <state_interface name="effort"/>
         </joint>
     </ros2_control>

Commit message: Refactor PropArm Hardware Interface and Propeller Force Controller
- Updated PropArmHardware to improve initialization and command handling.
- Enhanced PID controller parameters for better angle control.
- Adjusted motor speed limits and added gravity compensation logic.
- Refactored PropellerForceController to encapsulate methods and improve readability.
- Changed command interface limits in URDF to restrict position control range.
- Improved logging for better diagnostics and monitoring of control states.

File: prop_arm_description/models/prop_arm/urdf/prop_arm.urdf.xacro (robot description, xacro)
@@ -91,6 +91,6 @@
   <joint name="arm_link_joint" type="revolute">
     <axis xyz="0 0 -1"/>
-    <origin rpy="0 1.57080 0" xyz="0.43129 -0.58144 0.11764"/>
-    <limit lower="1.5708" upper="3.14159" effort="1500.0" velocity="10.0"/>
+    <origin rpy="-1.57080 0 -1.57080" xyz="0.43129 -0.58144 0.11764"/>
+    <limit lower="0" upper="1.5708" effort="1500.0" velocity="10.0"/>
     <dynamics damping="0.0" friction="0.0"/>
     <parent link="base_link"/>

File: prop_arm_gazebo_control/urdf/prop_arm_control.xacro (robot description, xacro)
@@ -29,6 +29,6 @@
             <!-- Command interface for position control (angle control) -->
             <command_interface name="position">
-                <param name="min">-3.14159</param>
-                <param name="max">3.14159</param>
+                <param name="min">0</param>
+                <param name="max">1.5708</param>
             </command_interface>
             <!-- State interfaces -->

Commit message: feat: Update aerospace data visualizer and control parameters for improved functionality

File: prop_arm_description/models/prop_arm/urdf/prop_arm.urdf.xacro (robot description, xacro)
@@ -6,18 +6,18 @@
   <link name="base_link">
     <collision name="base_collision">
-      <origin rpy="0.00000 0.00000 0.00000" xyz="0.00000 0.00000 0.00000"/>
+      <origin rpy="0 0 0" xyz="0 0 0"/>
       <geometry>
-        <mesh filename="package://prop_arm_description/models/prop_arm/meshes/collisions/base.stl" scale="1.00000 1.00000 1.00000"/>
+        <mesh filename="package://prop_arm_description/models/prop_arm/meshes/collisions/base.stl" scale="1 1 1"/>
       </geometry>
     </collision>
     <inertial>
-      <inertia ixx="4.49421" ixy="1.19011" ixz="-0.32403" iyy="1.83979" iyz="0.67570" izz="5.09395"/>
-      <origin rpy="0.00000 0.00000 0.00000" xyz="-0.00341 -0.01201 -0.10842"/>
-      <mass value="10.00000"/>
+      <inertia ixx="4.49421" ixy="0" ixz="0" iyy="1.83979" iyz="0" izz="5.09395"/>
+      <origin rpy="0 0 0" xyz="-0.00341 -0.01201 -0.10842"/>
+      <mass value="10.0"/>
     </inertial>
     <visual name="base">
-      <origin rpy="0.00000 0.00000 0.00000" xyz="0.00000 0.00000 0.00000"/>
+      <origin rpy="0 0 0" xyz="0 0 0"/>
       <geometry>
-        <mesh filename="package://prop_arm_description/models/prop_arm/meshes/visuals/base.dae" scale="1.00000 1.00000 1.00000"/>
+        <mesh filename="package://prop_arm_description/models/prop_arm/meshes/visuals/base.dae" scale="1 1 1"/>
       </geometry>
     </visual>
@@ -26,18 +26,18 @@
   <link name="arm_link">
     <collision name="arm_collision">
-      <origin rpy="0.00000 -1.57080 0.00000" xyz="0.00000 0.00000 -0.00000"/>
+      <origin rpy="0 -1.5708 0" xyz="0 0 0"/>
       <geometry>
-        <mesh filename="package://prop_arm_description/models/prop_arm/meshes/collisions/arm.stl" scale="1.00000 1.00000 1.00000"/>
+        <mesh filename="package://prop_arm_description/models/prop_arm/meshes/collisions/arm.stl" scale="1 1 1"/>
       </geometry>
     </collision>
     <inertial>
-      <inertia ixx="0.9156" ixy="-0.00006" ixz="-0.01066" iyy="0.91818" iyz="-0.00628" izz="0.01020"/>
-      <origin rpy="0.00000 0.00000 0.00000" xyz="0.14437 -0.00020 0.01985"/>
-      <mass value="20.0"/>
+      <inertia ixx="1.0e-05" ixy="0" ixz="0" iyy="2.7e-04" iyz="0" izz="2.7e-04"/>
+      <origin rpy="0 0 0" xyz="0.14437 -0.00020 0.01985"/>
+      <mass value="0.02"/>
     </inertial>
     <visual name="arm">
-      <origin rpy="0.00000 -1.57080 0.00000" xyz="0.00000 -0.00000 -0.00000"/>
+      <origin rpy="0 -1.5708 0" xyz="0 0 0"/>
       <geometry>
-        <mesh filename="package://prop_arm_description/models/prop_arm/meshes/visuals/arm.dae" scale="1.00000 1.00000 1.00000"/>
+        <mesh filename="package://prop_arm_description/models/prop_arm/meshes/visuals/arm.dae" scale="1 1 1"/>
       </geometry>
     </visual>
@@ -46,18 +46,18 @@
   <link name="motor_link">
     <collision name="motor_collision">
-      <origin rpy="0.00000 0.00000 0.00000" xyz="-0.00000 -0.00000 0.00000"/>
+      <origin rpy="0 0 0" xyz="0 0 0"/>
       <geometry>
-        <mesh filename="package://prop_arm_description/models/prop_arm/meshes/collisions/motor.stl" scale="1.00000 1.00000 1.00000"/>
+        <mesh filename="package://prop_arm_description/models/prop_arm/meshes/collisions/motor.stl" scale="1 1 1"/>
       </geometry>
     </collision>
     <inertial>
-      <inertia ixx="0.00229" ixy="0.00020" ixz="-0.00002" iyy="0.00144" iyz="0.00012" izz="0.00226"/>
-      <origin rpy="0.00000 0.00000 0.00000" xyz="-0.00013 0.00073 -0.00279"/>
-      <mass value="10.00000"/>
+      <inertia ixx="1.8825e-05" ixy="0" ixz="0" iyy="1.8825e-05" iyz="0" izz="1.5619e-05"/>
+      <origin rpy="0 0 0" xyz="-0.00013 0.00073 -0.00279"/>
+      <mass value="0.102"/>
     </inertial>
     <visual name="motor">
-      <origin rpy="0.00000 0.00000 0.00000" xyz="0.00000 0.00000 0.00000"/>
+      <origin rpy="0 0 0" xyz="0 0 0"/>
       <geometry>
-        <mesh filename="package://prop_arm_description/models/prop_arm/meshes/visuals/motor.dae" scale="1.00000 1.00000 1.00000"/>
+        <mesh filename="package://prop_arm_description/models/prop_arm/meshes/visuals/motor.dae" scale="1 1 1"/>
       </geometry>
     </visual>
@@ -66,18 +66,18 @@
   <link name="prop_link">
     <collision name="prop_collision">
-      <origin rpy="-0.00000 0.00000 0.00000" xyz="0.00000 0.00000 0.00000"/>
+      <origin rpy="0 0 0" xyz="0 0 0"/>
       <geometry>
-        <mesh filename="package://prop_arm_description/models/prop_arm/meshes/collisions/prop.stl" scale="1.00000 1.00000 1.00000"/>
+        <mesh filename="package://prop_arm_description/models/prop_arm/meshes/collisions/prop.stl" scale="1 1 1"/>
       </geometry>
     </collision>
     <inertial>
-      <inertia ixx="0.00022" ixy="-0.00077" ixz="-0.00002" iyy="0.03639" iyz="0.00000" izz="0.03655"/>
-      <origin rpy="0.00000 0.00000 0.00000" xyz="0.00007 0.00056 0.00001"/>
-      <mass value="10.00000"/>
+      <inertia ixx="1.0e-06" ixy="0" ixz="0" iyy="1.0e-06" iyz="0" izz="1.0e-06"/>
+      <origin rpy="0 0 0" xyz="0.00007 0.00056 0.00001"/>
+      <mass value="0.005"/>
     </inertial>
     <visual name="prop">
-      <origin rpy="0.00000 0.00000 0.00000" xyz="-0.00000 -0.00000 0.00000"/>
+      <origin rpy="0 0 0" xyz="0 0 0"/>
       <geometry>
-        <mesh filename="package://prop_arm_description/models/prop_arm/meshes/visuals/prop.dae" scale="1.00000 1.00000 1.00000"/>
+        <mesh filename="package://prop_arm_description/models/prop_arm/meshes/visuals/prop.dae" scale="1 1 1"/>
       </geometry>
     </visual>
