Commit message: New Upload

File: prop_arm_description/models/prop_arm_v2/urdf/prop_arm.urdf.xacro (robot description, xacro)
@@ -13,7 +13,5 @@
     <inertial>
       <mass value="2.343"/>
-      <inertia ixx="0.24075" ixy="-0.00000" ixz="0.00000"
-               iyy="0.23379" iyz="0.03671"
-               izz="0.01482"/>
+      <inertia ixx="0.24075" ixy="-0.00000" ixz="0.00000" iyy="0.23379" iyz="0.03671" izz="0.01482"/>
       <origin rpy="0.00000 0.00000 0.00000" xyz="-0.00883 0.00000 0.19143"/>
     </inertial>
@@ -35,7 +33,5 @@
     <inertial>
       <mass value="0.402"/>
-      <inertia ixx="0.00050" ixy="-0.00000" ixz="0.00129"
-               iyy="0.02111" iyz="-0.00000"
-               izz="0.02133"/>
+      <inertia ixx="0.00050" ixy="-0.00000" ixz="0.00129" iyy="0.02111" iyz="-0.00000" izz="0.02133"/>
       <origin rpy="0.00000 0.00000 0.00000" xyz="-0.19518 -0.00011 0.03646"/>
     </inertial>
@@ -57,7 +53,5 @@
     <inertial>
       <mass value="0.020"/>
-      <inertia ixx="0.00000043" ixy="0.00000194" ixz="0.00000000"
-               iyy="0.00007266" iyz="-0.00000000"
-               izz="0.00007301"/>
+      <inertia ixx="0.00000043" ixy="0.00000194" ixz="0.00000000" iyy="0.00007266" iyz="-0.00000000" izz="0.00007301"/>
       <origin rpy="0.00000 0.00000 0.00000" xyz="0.00000 0.00000 0.00454"/>
     </inertial>
@@ -78,5 +72,5 @@
     <axis xyz="0 1 0"/>
     <origin rpy="0 -1.57080 -1.57080" xyz="0.00001 -0.00000 0.45833"/>
-    <limit lower="-3.1416" upper="3.1416" effort="1500.0" velocity="10.0"/>
+    <limit lower="0.1421" upper="3.1416" effort="1500.0" velocity="10.0"/>
     <dynamics damping="0.0" friction="0.0"/>
     <parent link="base_link"/>

File: prop_arm_gazebo_control/urdf/prop_arm_control.xacro (robot description, xacro)
@@ -29,4 +29,10 @@
             <state_interface name="position"/>
             <state_interface name="velocity"/>
+            <state_interface name="position">
+                <param name="initial_value">0.1410</param>
+            </state_interface>
+            <state_interface name="velocity">
+                <param name="initial_value">0.0</param>
+            </state_interface>
         </joint>
     </ros2_control>

Commit message: feat: Enhance PropArm GUI with new control features and visualization charts
- Updated MainWindow to include new control panels for PWM input and step tests.
- Added three new charts for real-time visualization: Angle vs Reference, Tracking Error, and Motor Velocity.
- Implemented step test functionality with adjustable parameters for angle and timing.
- Improved UI elements for better user experience, including button labels and layout adjustments.
- Refactored data handling in PropArmGuiNode to support new simulation data and commands.
- Enhanced signal connections for automatic mode toggling and data updates.

File: prop_arm_description/models/prop_arm_v2/urdf/prop_arm.urdf.xacro (robot description, xacro)
@@ -72,5 +72,5 @@
     <axis xyz="0 1 0"/>
     <origin rpy="0 -1.57080 -1.57080" xyz="0.00001 -0.00000 0.45833"/>
-    <limit lower="0.1421" upper="3.1416" effort="1500.0" velocity="10.0"/>
+    <limit lower="0.16643634279943126" upper="3.1416" effort="1500.0" velocity="10.0"/>
     <dynamics damping="0.0" friction="0.0"/>
     <parent link="base_link"/>

File: prop_arm_gazebo_control/urdf/prop_arm_control.xacro (robot description, xacro)
@@ -30,5 +30,5 @@
             <state_interface name="velocity"/>
             <state_interface name="position">
-                <param name="initial_value">0.1410</param>
+                <param name="initial_value">0.16643634279943126</param>
             </state_interface>
             <state_interface name="velocity">

Commit message: Refactor PropArmHardware interface and remove step test input node
- Updated the PropArmHardware class to improve initialization, lifecycle management, and read/write cycles.
- Enhanced motor speed model integration and added support for PWM command handling.
- Removed the step_test_input_node.cpp file as it is no longer needed.
- Adjusted parameters in the URDF files for prop_arm_control and prop_arm_gazebo_plugins.
- Improved GUI code for better readability and maintainability, including updates to control data handling and chart updates.

File: prop_arm_description/models/prop_arm_v2/urdf/prop_arm.urdf.xacro (robot description, xacro)
@@ -32,7 +32,7 @@
     </collision>
     <inertial>
-      <mass value="0.402"/>
-      <inertia ixx="0.00050" ixy="-0.00000" ixz="0.00129" iyy="0.02111" iyz="-0.00000" izz="0.02133"/>
-      <origin rpy="0.00000 0.00000 0.00000" xyz="-0.19518 -0.00011 0.03646"/>
+      <mass value="0.4067"/>
+      <inertia ixx="0.00100" ixy="0.00000" ixz="0.00000" iyy="0.01086" iyz="0.00000" izz="0.01086"/>
+      <origin rpy="0.00000 0.00000 0.00000" xyz="-0.32745 -0.00011 0.03646"/>
     </inertial>
     <visual name="arm">
@@ -52,6 +52,6 @@
     </collision>
     <inertial>
-      <mass value="0.020"/>
-      <inertia ixx="0.00000043" ixy="0.00000194" ixz="0.00000000" iyy="0.00007266" iyz="-0.00000000" izz="0.00007301"/>
+      <mass value="0.0153"/>
+      <inertia ixx="0.00000033" ixy="0.00000148" ixz="0.00000000" iyy="0.00005558" iyz="-0.00000000" izz="0.00005585"/>
       <origin rpy="0.00000 0.00000 0.00000" xyz="0.00000 0.00000 0.00454"/>
     </inertial>
@@ -73,5 +73,5 @@
     <origin rpy="0 -1.57080 -1.57080" xyz="0.00001 -0.00000 0.45833"/>
     <limit lower="0.16643634279943126" upper="3.1416" effort="1500.0" velocity="10.0"/>
-    <dynamics damping="0.0" friction="0.0"/>
+    <dynamics damping="0.0326233" friction="0.0"/>
     <parent link="base_link"/>
     <child link="arm_link"/>

File: prop_arm_gazebo_control/urdf/prop_arm_control.xacro (robot description, xacro)
@@ -15,13 +15,15 @@
             <param name="actuator_index">0</param>
             <param name="prop_radius_m">0.1</param>
-            <param name="Kw">1.6975</param>
-            <param name="tau_w">0.500479</param>
+            <param name="Kw">1.4016</param>
+            <param name="tau_w">0.564</param>
+            <param name="L_w">0.294</param>
             <param name="Ts">0.01</param>
             <param name="pwm_ref_us">1000</param>
             <param name="pwm_max_us">2000</param>
             <param name="pwm_min_us">1000</param>
+            <param name="motor_cmd_scale">1.162</param>
         </hardware>
         <joint name="arm_link_joint">
-            <command_interface name="velocity">
+            <command_interface name="effort">
                 <param name="min">0.0</param>
                 <param name="max">750.0</param>

File: prop_arm_gazebo_plugins/urdf/prop_arm_gazebo_plugins.xacro (robot description, xacro)
@@ -11,11 +11,10 @@
             <timeConstantDown>0.0125</timeConstantDown>
             <maxRotVelocity>1178.0</maxRotVelocity>
-            <motorConstant>6.12e-06</motorConstant>
-            <momentConstant>1.224e-07</momentConstant>
+            <motorConstant>7.11e-06</motorConstant>
             <commandSubTopic>command/motor_speed</commandSubTopic>
             <actuator_number>0</actuator_number>
             <motorSpeedPubTopic>motor_speed/0</motorSpeedPubTopic>
             <rotorDragCoefficient>8.28e-05</rotorDragCoefficient>
-            <rollingMomentCoefficient>8.28e-06</rollingMomentCoefficient>
+            <rollingMomentCoefficient>1.00e-05</rollingMomentCoefficient>
             <rotorVelocitySlowdownSim>1</rotorVelocitySlowdownSim>
             <motorType>velocity</motorType>

Commit message: Add new widgets for telemetry visualization and export functionality
- Implement DutyPlot for visualizing duty cycle data with adjustable limits.
- Create ErrorPlot to display the absolute error between real and simulated angles.
- Introduce ExportPreviewDialog for previewing and exporting telemetry data to CSV.
- Add HoverChartView to enhance chart interaction with hover capabilities.
- Develop Panel widget for structured layout with a title.
- Implement PwmPlot for visualizing PWM signal data.
- Create SectionHeader for better organization of UI sections.
- Add SpeedPlot to visualize motor tip speed in real-time.
- Implement TrackingErrorPlot to visualize tracking errors between reference and actual angles.
- Create ValueTile for displaying labeled values with units in a compact format.

File: prop_arm_description/models/prop_arm_v2/urdf/prop_arm.urdf.xacro (robot description, xacro)
@@ -1,7 +1,22 @@
 <?xml version="1.0" encoding="utf-8"?>
 <robot xmlns:xacro="http://www.ros.org/wiki/xacro" name="prop_arm">
+  <!-- Load physics-only parameters -->
+  <xacro:arg name="physics_file" default="$(find-pkg-share prop_arm_description)/config/dynamics_params.xacro.yaml"/>
+  <!-- Convenience aliases -->
+  <xacro:property name="RAW" value="${xacro.load_yaml('$(arg physics_file)')}"/>
+  <xacro:property name="P" value="${RAW['prop_arm_description']['ros__parameters']}"/>
+  <xacro:property name="L" value="${P['links']}"/>
+  <xacro:property name="J" value="${P['joints']}"/>
+  <!-- Helper macro to reduce repetition -->
+  <xacro:macro name="inertial_from_yaml" params="link_name">
+    <inertial>
+      <mass value="${L[link_name]['mass']}"/>
+      <inertia ixx="${L[link_name]['inertia'][0]}" ixy="${L[link_name]['inertia'][1]}" ixz="${L[link_name]['inertia'][2]}" iyy="${L[link_name]['inertia'][3]}" iyz="${L[link_name]['inertia'][4]}" izz="${L[link_name]['inertia'][5]}"/>
+      <origin rpy="0 0 0" xyz="${L[link_name]['com_xyz'][0]} ${L[link_name]['com_xyz'][1]} ${L[link_name]['com_xyz'][2]}"/>
+    </inertial>
+  </xacro:macro>
   <!-- World link -->
   <link name="world"/>
-  <!-- Main robot link -->
+  <!-- Base link -->
   <link name="base_link">
     <collision name="base_collision">
@@ -11,9 +26,5 @@
       </geometry>
     </collision>
-    <inertial>
-      <mass value="2.343"/>
-      <inertia ixx="0.24075" ixy="-0.00000" ixz="0.00000" iyy="0.23379" iyz="0.03671" izz="0.01482"/>
-      <origin rpy="0.00000 0.00000 0.00000" xyz="-0.00883 0.00000 0.19143"/>
-    </inertial>
+    <xacro:inertial_from_yaml link_name="base_link"/>
     <visual name="base">
       <origin rpy="0 0 0" xyz="0 0 0"/>
@@ -31,9 +42,5 @@
       </geometry>
     </collision>
-    <inertial>
-      <mass value="0.4067"/>
-      <inertia ixx="0.00100" ixy="0.00000" ixz="0.00000" iyy="0.01086" iyz="0.00000" izz="0.01086"/>
-      <origin rpy="0.00000 0.00000 0.00000" xyz="-0.32745 -0.00011 0.03646"/>
-    </inertial>
+    <xacro:inertial_from_yaml link_name="arm_link"/>
     <visual name="arm">
       <origin rpy="0 0 0" xyz="0 0 0"/>
@@ -43,5 +50,5 @@
     </visual>
   </link>
-  <!-- Propeller link-->
+  <!-- Propeller link -->
   <link name="prop_link">
     <collision name="prop_collision">
@@ -51,9 +58,5 @@
       </geometry>
     </collision>
-    <inertial>
-      <mass value="0.0153"/>
-      <inertia ixx="0.00000033" ixy="0.00000148" ixz="0.00000000" iyy="0.00005558" iyz="-0.00000000" izz="0.00005585"/>
-      <origin rpy="0.00000 0.00000 0.00000" xyz="0.00000 0.00000 0.00454"/>
-    </inertial>
+    <xacro:inertial_from_yaml link_name="prop_link"/>
     <visual name="prop">
       <origin rpy="0 0 0" xyz="0 0 0"/>
@@ -72,6 +75,6 @@
     <axis xyz="0 1 0"/>
     <origin rpy="0 -1.57080 -1.57080" xyz="0.00001 -0.00000 0.45833"/>
-    <limit lower="0.16643634279943126" upper="3.1416" effort="1500.0" velocity="10.0"/>
-    <dynamics damping="0.0326233" friction="0.0"/>
+    <limit lower="${J['arm_link_joint']['limit_lower']}" upper="${J['arm_link_joint']['limit_upper']}" effort="${J['arm_link_joint']['effort']}" velocity="${J['arm_link_joint']['velocity']}"/>
+    <dynamics damping="${J['arm_link_joint']['damping']}" friction="${J['arm_link_joint']['friction']}"/>
     <parent link="base_link"/>
     <child link="arm_link"/>

File: prop_arm_gazebo_control/urdf/prop_arm_control.xacro (robot description, xacro)
@@ -1,4 +1,13 @@
 <?xml version="1.0"?>
 <robot xmlns:xacro="http://www.ros.org/wiki/xacro" name="prop_arm_control">
+    <!-- Load physics-only parameters -->
+    <xacro:arg name="motor_config" default="$(find prop_arm_gazebo_control)/config/motor_model.yaml"/>
+    <!-- Convenience aliases -->
+    <xacro:property name="RAW" value="${xacro.load_yaml('$(arg motor_config)')}"/>
+    <xacro:property name="P" value="${RAW['prop_arm_gazebo_control']['ros__parameters']}"/>
+    <xacro:property name="MM" value="${P['motor_model']}"/>
+    <xacro:property name="CTRL" value="${P['control']}"/>
+    <xacro:property name="RC" value="${P['ros2_control']}"/>
+    <!-- GZ ROS2 control plugin -->
     <gazebo>
         <plugin filename="gz_ros2_control-system" name="gz_ros2_control::GazeboSimROS2ControlPlugin">
@@ -11,29 +20,31 @@
         <hardware>
             <plugin>prop_arm_gazebo_control/PropArmHardware</plugin>
-            <param name="robot_namespace">arm_sim</param>
-            <param name="joint_name">arm_link_joint</param>
-            <param name="actuator_index">0</param>
-            <param name="prop_radius_m">0.1</param>
-            <param name="Kw">1.4016</param>
-            <param name="tau_w">0.564</param>
-            <param name="L_w">0.294</param>
-            <param name="Ts">0.01</param>
-            <param name="pwm_ref_us">1000</param>
-            <param name="pwm_max_us">2000</param>
-            <param name="pwm_min_us">1000</param>
-            <param name="motor_cmd_scale">1.162</param>
+            <param name="robot_namespace">${RC['robot_namespace']}</param>
+            <param name="joint_name">${RC['joint_name']}</param>
+            <param name="actuator_index">${RC['actuator_index']}</param>
+            <param name="prop_radius_m">${MM['prop_radius_m']}</param>
+            <param name="c1">${MM['c1']}</param>
+            <param name="c2">${MM['c2']}</param>
+            <param name="d1">${MM['d1']}</param>
+            <param name="d2">${MM['d2']}</param>
+            <param name="L_w">${MM['L_w']}</param>
+            <param name="Ts">${MM['Ts']}</param>
+            <param name="pwm_min_us">${MM['pwm_min_us']}</param>
+            <param name="pwm_max_us">${MM['pwm_max_us']}</param>
+            <param name="motor_cmd_scale">${MM['motor_cmd_scale']}</param>
+            <param name="pwm_spin_min_us">${MM['pwm_spin_min_us']}</param>
         </hardware>
         <joint name="arm_link_joint">
             <command_interface name="effort">
-                <param name="min">0.0</param>
-                <param name="max">750.0</param>
+                <param name="min">${CTRL['command_effort_min']}</param>
+                <param name="max">${CTRL['command_effort_max']}</param>
             </command_interface>
             <state_interface name="position"/>
             <state_interface name="velocity"/>
             <state_interface name="position">
-                <param name="initial_value">0.16643634279943126</param>
+                <param name="initial_value">${CTRL['initial_position']}</param>
             </state_interface>
             <state_interface name="velocity">
-                <param name="initial_value">0.0</param>
+                <param name="initial_value">${CTRL['initial_velocity']}</param>
             </state_interface>
         </joint>
